File: hardware/rev_a/MainAutobike.brd (EAGLE design)
At the start: 127 x 101.6 mm, 138 parts, among them J13 TC2030-CTX, U1 ATUM, U2 PCA9685, U3 PCA9685, U4 ADXL362

Commit message: updated pcb, added pdfs
Routing:
- net N$31: track 12.3 -> 16.5 mm
- net N$20: track 12.3 -> 16.5 mm
- net AIN6: track 21.5 -> 25.1 mm
- net N$27: track 13.3 -> 16.5 mm
- net P22: track 20.1 -> 22.6 mm
- net GND: vias 1 -> 11

Commit message: charles, look over hall effect please; checked rest of schematic and board
Parts:
- added U$3: (no value), logos:UMICH_SOLID_75MIL
Other:
- board text added: "D"
- board text added: "D.A., C.H., T.K., K.S., A.Z."
- board text added: "I"
- board text added: "L"
- board text added: "R"
- board text added: "SCL"
- board text added: "SDA"
Changed lines of the file:
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@@
 <wire x1="-16.256" y1="12.446" x2="-16.256" y2="16.002" width="0.3048" layer="21"/>
 <text x="-15.621" y="13.462" size="1.778" layer="21" ratio="12">A</text>
+<wire x1="-58.928" y1="-60.198" x2="-57.658" y2="-60.198" width="0.254" layer="21"/>
+<wire x1="-57.658" y1="-60.198" x2="-57.658" y2="-61.976" width="0.254" layer="21"/>
+<wire x1="-57.658" y1="-61.976" x2="-58.928" y2="-61.976" width="0.254" layer="21"/>
+<wire x1="-58.928" y1="-61.976" x2="-58.928" y2="-60.198" width="0.254" layer="21"/>
+<text x="-58.5597" y="-61.468" size="0.8128" layer="21" ratio="12">A</text>
+<text x="57.658" y="-62.738" size="0.7112" layer="21" ratio="12">D.A., C.H.,
+T.K., K.S.,
+A.Z.</text>
+<text x="-6.604" y="29.464" size="0.7112" layer="21" ratio="12" rot="R90">SCL</text>
+<text x="-6.604" y="32.512" size="0.7112" layer="21" ratio="12" rot="R90">SDA</text>
+<text x="11.938" y="-61.976" size="0.7112" layer="21" ratio="12">SDA</text>
+<text x="9.144" y="-61.976" size="0.7112" layer="21" ratio="12">SCL</text>
+<text x="29.21" y="-58.42" size="0.7112" layer="21" ratio="12">L</text>
+<text x="26.416" y="-58.42" size="0.7112" layer="21" ratio="12">R</text>
+<text x="23.876" y="-58.42" size="0.7112" layer="21" ratio="12">I</text>
+<text x="21.336" y="-58.42" size="0.7112" layer="21" ratio="12">D</text>
 </plain>
 <attributes>
@@
 <element name="GLED1" library="led" package="CHIP-LED0603" value="" x="38.1" y="-50.8"/>
 <element name="GLED2" library="led" package="CHIP-LED0603" value="" x="-38.1" y="-50.8"/>
-<element name="RLED1" library="led" package="CHIP-LED0603" value="" x="-17.78" y="-43.18"/>
-<element name="RLED2" library="led" package="CHIP-LED0603" value="" x="-12.7" y="-43.18"/>
-<element name="RLED3" library="led" package="CHIP-LED0603" value="" x="-7.62" y="-43.18"/>
-<element name="RLED4" library="led" package="CHIP-LED0603" value="" x="-2.54" y="-43.18"/>
-<element name="RLED5" library="led" package="CHIP-LED0603" value="" x="2.54" y="-43.18"/>
-<element name="RLED6" library="led" package="CHIP-LED0603" value="" x="7.62" y="-43.18"/>
-<element name="RLED7" library="led" package="CHIP-LED0603" value="" x="12.7" y="-43.18"/>
-<element name="RLED8" library="led" package="CHIP-LED0603" value="" x="17.78" y="-43.18"/>
+<element name="RLED1" library="led" package="CHIP-LED0603" value="" x="-17.78" y="-43.18" smashed="yes">
+<attribute name="NAME" x="-18.415" y="-44.831" size="1.27" layer="25" rot="R90"/>
+<attribute name="VALUE" x="-15.875" y="-43.815" size="1.27" layer="27" rot="R90"/>
+</element>
+<element name="RLED2" library="led" package="CHIP-LED0603" value="" x="-12.7" y="-43.18" smashed="yes">
+<attribute name="NAME" x="-13.335" y="-44.831" size="1.27" layer="25" rot="R90"/>
+<attribute name="VALUE" x="-10.795" y="-43.815" size="1.27" layer="27" rot="R90"/>
+</element>
+<element name="RLED3" library="led" package="CHIP-LED0603" value="" x="-7.62" y="-43.18" smashed="yes">
+<attribute name="NAME" x="-8.255" y="-44.831" size="1.27" layer="25" rot="R90"/>
+<attribute name="VALUE" x="-5.715" y="-43.815" size="1.27" layer="27" rot="R90"/>
+</element>
+<element name="RLED4" library="led" package="CHIP-LED0603" value="" x="-2.54" y="-43.18" smashed="yes">
+<attribute name="NAME" x="-3.175" y="-44.831" size="1.27" layer="25" rot="R90"/>
+<attribute name="VALUE" x="-0.635" y="-43.815" size="1.27" layer="27" rot="R90"/>
+</element>
+<element name="RLED5" library="led" package="CHIP-LED0603" value="" x="2.54" y="-43.18" smashed="yes">
+<attribute name="NAME" x="1.905" y="-44.831" size="1.27" layer="25" rot="R90"/>
+<attribute name="VALUE" x="4.445" y="-43.815" size="1.27" layer="27" rot="R90"/>
+</element>
+<element name="RLED6" library="led" package="CHIP-LED0603" value="" x="7.62" y="-43.18" smashed="yes">
+<attribute name="NAME" x="6.985" y="-44.831" size="1.27" layer="25" rot="R90"/>
+<attribute name="VALUE" x="9.525" y="-43.815" size="1.27" layer="27" rot="R90"/>
+</element>
+<element name="RLED7" library="led" package="CHIP-LED0603" value="" x="12.7" y="-43.18" smashed="yes">
+<attribute name="NAME" x="11.811" y="-44.831" size="1.27" layer="25" rot="R90"/>
+<attribute name="VALUE" x="14.605" y="-43.815" size="1.27" layer="27" rot="R90"/>
+</element>
+<element name="RLED8" library="led" package="CHIP-LED0603" value="" x="17.78" y="-43.18" smashed="yes">
+<attribute name="NAME" x="17.145" y="-44.831" size="1.27" layer="25" rot="R90"/>
+<attribute name="VALUE" x="19.685" y="-43.815" size="1.27" layer="27" rot="R90"/>
+</element>
 <element name="U$12" library="25AA02E48" package="SOT23-6" value="25AA02E48-SOT-23-6" x="44.45" y="-12.7"/>
 <element name="U$13" library="25AA02E48" package="SOT23-6" value="25AA02E48-SOT-23-6" x="44.45" y="-31.75"/>
@@
 <element name="U$14" library="PJ063PH" package="PJ063BH" value="PJ063PH" x="-3.81" y="19.05" rot="R270"/>
 <element name="U$1" library="logos" package="UMICH_SOLID_200MIL" value="" x="-24.638" y="12.192"/>
+<element name="U$3" library="logos" package="UMICH_SOLID_75MIL" value="" x="-62.484" y="-61.976"/>
 </elements>
 <signals>

Commit message: final revision A of PCB
Parts:
- added DEC_GEAR_SWITCH1, INC_GEAR_SWITCH1: LED_SWITCH, led_switch:LED_SWITCH
- added GLED4: (no value), led:CHIP-LED0603
- added JP13, JP14, JP15, JP19, JP8: (no value), pinhead:1X04
- added JP16, JP17, JP18, JP20, JP9: (no value), pinhead:1X03
- added JP21, JP22: (no value), pinhead:1X02
- added R36, R45, R46, R47, R48: 10k, rcl:R0603
- added R37, R39, R41, R42, R49: 1k, rcl:R0603
- added R38, R40, R43, R44, R50: 390, rcl:R0603
- added R51, R52, R53, R54, R55, R56, R57, R58: 33, rcl:R0402
- added R59: 60.4, rcl:R0402
- added U$20, U$22, U$23, U$24, U$25, U$28, U$29, U$31, U$32, U$34: 25AA02E48-SOT-23-6, 25AA02E48:SOT23-3
- added U$21, U$26, U$27, U$30, U$33: HALLEFFECT, 25AA02E48:SOT23-6
- JP1, JP2, JP3: device pinhead:1X03 -> pinhead:1X04
- R1, R2: device microbuilder:0805 -> rcl:R0603
- R17, R18, R25: value 1k -> 10k
- U$12, U$13, U$15, U$16, U$17, U$19: device 25AA02E48:SOT23-6 -> 25AA02E48:SOT23-3
- moved U$17 44.9 mm to (28.7, 15.6), turned to 270 degrees
- moved JP3 44.5 mm to (18.4, 15.2), turned to 180 degrees
- moved R18 44.3 mm to (25.4, 15.1), turned to 0 degrees
- moved U$13 40.0 mm to (57.1, 6.22), turned to 90 degrees
- moved R21 35.4 mm to (57.1, 3.30), turned to 180 degrees
- moved JP12 33.9 mm to (61.0, 4.70), turned to 90 degrees
- moved U$6 32.9 mm to (53.5, 6.22)
- moved U$12 31.2 mm to (57.1, 15.7), turned to 90 degrees
- moved R24 28.2 mm to (53.5, 2.79), turned to 180 degrees
- moved R22 26.2 mm to (57.1, 13.0), turned to 180 degrees
- moved JP11 24.4 mm to (61.0, 14.2), turned to 90 degrees
- moved U$5 23.9 mm to (53.5, 15.7)
- moved U$16 19.7 mm to (28.7, 9.27), turned to 270 degrees
- moved JP2 19.1 mm to (18.4, 8.89), turned to 180 degrees
- moved R25 18.8 mm to (25.4, 8.64), turned to 0 degrees
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Connections:
- new net GND_LGT1: JP1.4, R17.1
- new net GND_LGT2: JP2.4, R25.1
- new net GND_LGT3: JP3.4, R18.1
- new net GND_LGT4: JP8.4, R36.1
- new net GND_LGT5: JP13.4, R45.1
- new net GND_LGT6: JP14.4, R47.1
- new net GND_LGT7: JP15.4, R46.1
- new net GND_LGT8: JP19.4, R48.1
- new net HE4GND: JP9.3, U$21.5, U$22.2
- new net HE4OUT: JP9.2, R38.1, U$22.3
- new net HE4VIN: JP9.1, R38.2, U$21.1
- new net HE5GND: JP16.3, U$30.5, U$31.2
- new net HE5OUT: JP16.2, R40.1, U$31.3
- new net HE5VIN: JP16.1, R40.2, U$30.1
- new net HE6GND: JP17.3, U$26.5, U$28.2
- new net HE6OUT: JP17.2, R43.1, U$28.3
- new net HE6VIN: JP17.1, R43.2, U$26.1
- new net HE7GND: JP18.3, U$27.5, U$29.2
- new net HE7OUT: JP18.2, R44.1, U$29.3
- new net HE7VIN: JP18.1, R44.2, U$27.1
- new net HE8GND: JP20.3, U$33.5, U$34.2
- new net HE8OUT: JP20.2, R50.1, U$34.3
- new net HE8VIN: JP20.1, R50.2, U$33.1
- new net N$19: R39.2, U$30.3
- new net N$22: R41.2, U$27.3
- new net N$33: JP8.3, R55.1
- new net N$34: JP3.3, R56.1
- new net N$39: JP2.3, R57.1
- new net N$42: JP1.3, R58.1
- new net N$43: INC_GEAR_SWITCH1.P$4, JP21.2
- new net N$44: INC_GEAR_SWITCH1.P$2, JP21.1
- new net N$45: DEC_GEAR_SWITCH1.P$4, JP22.2
- new net N$49: DEC_GEAR_SWITCH1.P$2, JP22.1
- new net N$79: GLED4.A, R59.1
- new net OUT_LGT1: R17.2, R58.2, U$15.2
- new net OUT_LGT2: R25.2, R57.2, U$16.2
- new net OUT_LGT3: R18.2, R56.2, U$17.2
- new net OUT_LGT4: R36.2, R55.2, U$20.2
- new net OUT_LGT5: R45.2, R54.2, U$23.2
- new net OUT_LGT6: R47.2, R53.2, U$24.2
- new net OUT_LGT7: R46.2, R52.2, U$25.2
- new net OUT_LGT8: R48.2, R51.2, U$32.2
- new net SIG_LGT1: JP1.2, U$15.1
- new net SIG_LGT2: JP2.2, U$16.1
- new net SIG_LGT3: JP3.2, U$17.1
- new net SIG_LGT4: JP8.2, U$20.1
- new net SIG_LGT5: JP13.2, U$23.1
- new net SIG_LGT6: JP14.2, U$24.1
- new net SIG_LGT7: JP15.2, U$25.1
- new net SIG_LGT8: JP19.2, U$32.1
- new net VCC_LGT1: JP1.1, U$15.3
- new net VCC_LGT2: JP2.1, U$16.3
- new net VCC_LGT3: JP3.1, U$17.3
- new net VCC_LGT4: JP8.1, U$20.3
- new net VCC_LGT5: JP13.1, U$23.3
- new net VCC_LGT6: JP14.1, U$24.3
- new net VCC_LGT7: JP15.1, U$25.3
- new net VCC_LGT8: JP19.1, U$32.3
- net HE1GND: now also U$19.2; no longer U$19.4
- net HE1OUT: now also U$19.3; no longer U$19.1, U$19.2, U$19.5, U$19.6
- net HE2GND: now also U$12.2; no longer U$12.4
- net HE2OUT: now also U$12.3; no longer U$12.1, U$12.2, U$12.5, U$12.6
- net HE3GND: now also U$13.2; no longer U$13.4
- net HE3OUT: now also U$13.3; no longer U$13.1, U$13.2, U$13.5, U$13.6
- net N$13: now also R37.1, U$22.1; no longer JP1.2, R17.1
- net N$14: now also R37.2, U$21.3; no longer R17.2, U$15.3
- net N$15: now also U$19.1; no longer U$19.3
- net N$17: now also R39.1, U$31.1; no longer JP1.3, U$15.4
- net N$18: now also U$13.1; no longer U$13.3
- net N$20: now also R41.1, U$29.1; no longer JP1.1, U$15.1, U$15.2, U$15.5, U$15.6
- net N$23: now also R42.1, U$28.1; no longer JP2.2, R25.1
- net N$24: now also U$12.1; no longer U$12.3
- net N$26: now also R42.2, U$26.3; no longer R25.2, U$16.3
- net N$27: now also R49.1, U$34.1; no longer JP2.1, U$16.1, U$16.2, U$16.5, U$16.6
- net N$28: now also R49.2, U$33.3; no longer JP2.3, U$16.4
- net N$29: now also JP19.3, R51.1; no longer JP3.2, R18.1
- net N$30: now also JP15.3, R52.1; no longer R18.2, U$17.3
- net N$31: now also JP14.3, R53.1; no longer JP3.1, U$17.1, U$17.2, U$17.5, U$17.6
- net N$32: now also JP13.3, R54.1; no longer JP3.3, U$17.4
- net VCC(3.3V): now also R59.2
Routing:
- net VCC(3.3V): track 287.6 -> 314.5 mm, vias 4 -> 6
- net HE2GND: track 26.0 -> 8.93 mm, vias 3 -> 0
- net HE3GND: track 25.7 -> 8.93 mm, vias 3 -> 0
- net HE2OUT: track 29.8 -> 13.3 mm, vias 1 -> 2
- net HE3OUT: track 29.6 -> 13.5 mm, vias 1 -> 2
- net OUT_LGT1: track 0.00 -> 15.8 mm
- net HE1GND: track 24.5 -> 8.83 mm, vias 3 -> 0
- net OUT_LGT7: track 0.00 -> 15.3 mm
- net OUT_LGT8: track 0.00 -> 15.3 mm
- net OUT_LGT5: track 0.00 -> 15.2 mm
- net OUT_LGT3: track 0.00 -> 15.2 mm
- net OUT_LGT6: track 0.00 -> 15.1 mm
- net OUT_LGT2: track 0.00 -> 15.1 mm
- net OUT_LGT4: track 0.00 -> 15.0 mm
- net N$31: track 16.5 -> 2.04 mm
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- added copper zone on layer 1, net GND_LGT1
- added copper zone on layer 16, net GND_LGT1
- added copper zone on layer 1, net GND_LGT2
- added copper zone on layer 16, net GND_LGT2
- added copper zone on layer 1, net GND_LGT3
- added copper zone on layer 16, net GND_LGT3
- added copper zone on layer 1, net GND_LGT4
- added copper zone on layer 16, net GND_LGT4
- added copper zone on layer 1, net GND_LGT5
- added copper zone on layer 16, net GND_LGT5
- added copper zone on layer 1, net GND_LGT6
- added copper zone on layer 16, net GND_LGT6
- added copper zone on layer 1, net GND_LGT7
- added copper zone on layer 16, net GND_LGT7
- added copper zone on layer 1, net GND_LGT8
- added copper zone on layer 16, net GND_LGT8
- removed copper zone on layer 1, net N$42
- removed copper zone on layer 16, net N$43
- removed copper zone on layer 16, net N$44
- removed copper zone on layer 1, net N$45
- removed copper zone on layer 16, net N$49
- removed copper zone on layer 1, net N$50
- removed copper zone on layer 1, net N$51
- removed copper zone on layer 16, net N$52
Other:
- outline, holes or cut-outs redrawn

Commit message: crap...
Connections:
- net GND: now also GLED4.C
Changed lines of the file:
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@@
 <?xml version="1.0" encoding="utf-8"?>
 <!DOCTYPE eagle SYSTEM "eagle.dtd">
-<eagle version="6.6.0">
+<eagle version="6.4">
 <drawing>
 <settings>
@@
 <via x="-38.354" y="1.27" extent="1-16" drill="0.5"/>
 <via x="-41.402" y="-32.004" extent="1-16" drill="0.5"/>
+<contactref element="GLED4" pad="C"/>
 </signal>
 <signal name="TDO">
@@
 </signal>
 </signals>
-<errors>
-</errors>
 </board>
 </drawing>
